Commit message: fixed robotiq 85 gripper model

File: urdf/robot.urdf.xacro (robot description, xacro)
@@ -19,5 +19,5 @@
        - hardware_interface/VelocityJointInterface
        - hardware_interface/EffortJointInterface
--->
+  -->
   <xacro:arg name="transmission_hw_interface"
              default="hardware_interface/PositionJointInterface"/>
@@ -171,57 +171,31 @@
       <origin xyz="0.0 0.0 1" rpy="0.0 0.0 -1.5707963" />
    </joint>
-    <!-- End Effector -->
-    <joint name="ee_fixed_joint" type="fixed">
-        <parent link="wrist_3_link"/>
-        <child link="ee_link"/>
-        <origin rpy="0.0 0.0 1.57079632679" xyz="0.0 0.0823 0.0"/>
+    <link name="robotiq_85_gripper">
+      <visual>
+        <geometry>
+          <!-- The path to the visual meshes in the package. -->
+          <mesh filename="package://agimus_demos/ur3/pointing/meshes/gripper_2f85_opened.stl" scale = "0.0008 0.0008 0.0008" />
+        </geometry>
+      </visual>
+      <collision>
+        <geometry>
+          <!-- The path to the collision meshes in the package. -->
+          <mesh filename="package://agimus_demos/ur3/pointing/meshes/gripper_2f85_opened.stl" scale = "0.0008 0.0008 0.0008" />
+        </geometry>
+      </collision>
+    </link>
+    <joint name="robotiq_85_gripper_joint" type="fixed">
+      <!-- The parent link must be read from the robot model it is attached to. -->
+      <parent link="wrist_3_link"/>
+      <child link="robotiq_85_gripper"/>
+      <origin rpy="1.5708 0 0" xyz="0 0.075 0"/>
     </joint>
-    <link name="ee_link">
-    <collision>
-      <geometry>
-        <box size="0.01 0.01 0.01"/>
-      </geometry>
-      <origin rpy="0 0 0" xyz="-0.01 0 0"/>
-    </collision>
-    </link>
-  <!-- Robotiq Coupler -->
-  <!-- Gripper -->
-  <xacro:include filename="$(find agimus_demos)/ur3/pointing/urdf/robotiq_gripper/robotiq_85_gripper.urdf.xacro" />
-  <!--  + Height added by the coupler: 8mm -->
-  <!--  + Reference frame: at the middle (4mm) -->
-  <link name="robotiq_coupler">
-    <visual>
-      <geometry>
-        <mesh filename="package://agimus_demos/ur3/pointing/meshes/robotiq_85_coupler.stl" />
-      </geometry>
-      <material name="flat_black"/>
-    </visual>
-    <collision>
-      <geometry>
-        <mesh filename="package://agimus_demos/ur3/pointing/meshes/robotiq_85_coupler.stl" />
-      </geometry>
-    </collision>
-    <inertial>
-      <origin xyz="2.073e-05   1.45286e-03  -1.1049e-03" rpy="0 0 0" />
-      <mass value="0.168" />
-      <inertia ixx="6.69695624e-05" ixy="5.21511788e-09" ixz="-2.74383009e-08"
-               iyy="7.85088161e-05" iyz="5.41105193e-07" izz="1.41819717e-04"/>
-    </inertial>
-  </link>
-  <joint name="robotiq_coupler_joint" type="fixed">
-    <origin xyz="0 0 0.004" rpy="0 0 ${-pi/2.0}" />
-    <parent link="tool0"/>
-    <child link="robotiq_coupler"/>
-  </joint>
-  <gazebo reference="robotiq_coupler">
-    <mu1>0.9</mu1>
-    <mu2>0.9</mu2>
-    <material>Gazebo/FlatBlack</material>
-  </gazebo>
-  <!-- Attach the robotiq 85 gripper -->
-  <xacro:robotiq_85_gripper prefix="" parent="robotiq_coupler" >
-    <origin xyz="0 0 0.004" rpy="0 ${-pi/2} ${pi}"/>
-  </xacro:robotiq_85_gripper>
-   <!-- Camera -->
+    <!-- TCP frame -->
+    <joint name="tcp_joint" type="fixed">
+      <origin xyz="0 0 0.116" rpy="0 0 0"/>
+      <parent link="robotiq_85_gripper"/>
+      <child link="tcp"/>
+    </joint>
+    <link name="tcp"/>
    <link name="ref_camera_link">
    </link>

Commit message: Build control graph for UR3 demo

File: urdf/robot.urdf.xacro (robot description, xacro)
@@ -175,5 +175,5 @@
         <geometry>
           <!-- The path to the visual meshes in the package. -->
-          <mesh filename="package://agimus_demos/ur3/pointing/meshes/gripper_2f85_opened.stl" scale = "0.0008 0.0008 0.0008" />
+          <mesh filename="package://agimus_demos/ur3/pointing/meshes/gripper_2f85_opened.stl" scale = "0.001 0.001 0.001" />
         </geometry>
       </visual>
@@ -181,14 +181,38 @@
         <geometry>
           <!-- The path to the collision meshes in the package. -->
-          <mesh filename="package://agimus_demos/ur3/pointing/meshes/gripper_2f85_opened.stl" scale = "0.0008 0.0008 0.0008" />
+          <mesh filename="package://agimus_demos/ur3/pointing/meshes/gripper_2f85_opened.stl" scale = "0.001 0.001 0.001" />
         </geometry>
       </collision>
     </link>
-    <joint name="robotiq_85_gripper_joint" type="fixed">
-      <!-- The parent link must be read from the robot model it is attached to. -->
-      <parent link="wrist_3_link"/>
-      <child link="robotiq_85_gripper"/>
-      <origin rpy="1.5708 0 0" xyz="0 0.075 0"/>
-    </joint>
+    <link name="robotiq_coupler">
+    <visual>
+      <geometry>
+        <mesh filename="package://agimus_demos/ur3/pointing/meshes/robotiq_85_coupler.stl" />
+      </geometry>
+      <material name="flat_black"/>
+    </visual>
+    <collision>
+      <geometry>
+        <mesh filename="package://agimus_demos/ur3/pointing/meshes/robotiq_85_coupler.stl" />
+      </geometry>
+    </collision>
+    <inertial>
+      <origin xyz="2.073e-05   1.45286e-03  -1.1049e-03" rpy="0 0 0" />
+      <mass value="0.168" />
+      <inertia ixx="6.69695624e-05" ixy="5.21511788e-09" ixz="-2.74383009e-08"
+               iyy="7.85088161e-05" iyz="5.41105193e-07" izz="1.41819717e-04"/>
+    </inertial>
+  </link>
+  <joint name="robotiq_coupler_joint" type="fixed">
+    <origin xyz="0 0 0.004" rpy="0 0 ${-pi/2.0}" />
+    <parent link="tool0"/>
+    <child link="robotiq_coupler"/>
+  </joint>
+  <!-- Attach the robotiq 85 gripper -->
+   <joint name="robotiq_85_gripper_joint" type="fixed">
+     <parent link="robotiq_coupler"/>
+     <child link="robotiq_85_gripper"/>
+    <origin xyz="-0.09 0 0" rpy="${pi/2} 0 ${pi/2}"/>
+  </joint>
     <!-- TCP frame -->
     <joint name="tcp_joint" type="fixed">

Commit message: calibration realsense D435

File: urdf/robot.urdf.xacro (robot description, xacro)
@@ -85,18 +85,4 @@
     </link>
      <link name="walls">
-     <!-- front wall -->
-     <!-- visual -->
-	<!-- origin xyz="0.385 -0.305 0.37"/ -->
-        <!-- geometry -->
-	  <!-- box size="0.03 1 0.74"/ -->
-        <!-- /geometry -->
-	<!-- material name="white02"/ -->
-     <!-- /visual -->
-      <collision>
-       <origin xyz="0.385 -0.305 0.37"/>
-       <geometry>
-	 <box size="0.03 1 0.74"/>
-       </geometry>
-      </collision>
       <!-- behind wall -->
      <visual>
@@ -173,16 +159,16 @@
    <!-- Gripper -->
     <link name="robotiq_85_gripper">
-      <visual>
-        <geometry>
-          <!-- The path to the visual meshes in the package. -->
+     <!-- <visual>
+        <geometry>
+         The path to the visual meshes in the package.
           <mesh filename="package://agimus_demos/ur3/pointing/meshes/gripper_2f85_opened.stl" scale = "0.001 0.001 0.001" />
         </geometry>
-      </visual>
-      <collision>
-        <geometry>
-          <!-- The path to the collision meshes in the package. -->
+      </visual> -->
+      <!-- collision>
+        <geometry>
+          < The path to the collision meshes in the package. >
           <mesh filename="package://agimus_demos/ur3/pointing/meshes/gripper_2f85_opened.stl" scale = "0.001 0.001 0.001" />
         </geometry>
-      </collision>
+      </collision> -->
     </link>
     <link name="robotiq_coupler">
@@ -206,5 +192,5 @@
   </link>
   <joint name="robotiq_coupler_joint" type="fixed">
-    <origin xyz="0 0 0.004" rpy="0 0 ${-pi/2.0}" />
+    <origin xyz="0 0 0.01" rpy="0 0 ${-pi/2.0}" />
     <parent link="tool0"/>
     <child link="robotiq_coupler"/>
@@ -223,8 +209,38 @@
     </joint>
     <link name="tcp"/>
+    <!-- Camera -->
+    <link name="ur3_d435_mount_link">
+     <inertial>
+       <origin xyz="0.0 0.0 0.0" rpy="0 0 0" />
+       <mass value="0.1"/>
+       <inertia ixx="0.001" ixy="0.0" ixz="0.0"
+         iyy="0.001" iyz="0.0"
+         izz="0.001" />
+     </inertial>
+     <visual>
+       <origin xyz="0 0 0" rpy="0 0 0" />
+       <geometry>
+         <mesh filename="package://agimus_demos/ur3/pointing/meshes/ur3_d435_mount.stl"/>
+       </geometry>
+       <material name="Red">
+         <color rgba="0.9 0.1 0.1 1.0"/>
+       </material>
+     </visual>
+     <collision>
+       <origin xyz="0 0 0" rpy="0 0 0" />
+       <geometry>
+         <mesh filename="package://agimus_demos/ur3/pointing/meshes/ur3_d435_mount.stl"/>
+       </geometry>
+     </collision>
+   </link>
+   <joint name="ur3_d435_mount_joint" type="fixed">
+     <parent link="wrist_3_link"/>
+     <child link="ur3_d435_mount_link" />
+     <origin xyz="0.0 0.0 0.0" rpy="0.0 0.0 3.14159265359" />
+   </joint>
    <link name="ref_camera_link">
    </link>
     <joint name="ref_camera_joint" type="fixed">
-     <parent link="wrist_3_link" />
+     <parent link="ur3_d435_mount_link" />
      <child link = "ref_camera_link" />
      <origin xyz="${camera_pose['camera']['x']}

Commit message: update grasp and handle configurations for plaque-ur3

File: urdf/robot.urdf.xacro (robot description, xacro)
@@ -159,16 +159,14 @@
    <!-- Gripper -->
     <link name="robotiq_85_gripper">
-     <!-- <visual>
-        <geometry>
-         The path to the visual meshes in the package.
+     <visual>
+        <geometry>
           <mesh filename="package://agimus_demos/ur3/pointing/meshes/gripper_2f85_opened.stl" scale = "0.001 0.001 0.001" />
         </geometry>
-      </visual> -->
-      <!-- collision>
-        <geometry>
-          < The path to the collision meshes in the package. >
+      </visual>
+      <collision>
+        <geometry>
           <mesh filename="package://agimus_demos/ur3/pointing/meshes/gripper_2f85_opened.stl" scale = "0.001 0.001 0.001" />
         </geometry>
-      </collision> -->
+      </collision> >
     </link>
     <link name="robotiq_coupler">
@@ -256,3 +254,11 @@
       <origin xyz="0 0 0" rpy="0 0 0"/>
    </xacro:sensor_d435>
+      <!-- Axes -->
+      <link name="gripper_axe">
+      </link>
+       <joint name="gripper_axe_joint" type="fixed">
+        <origin xyz="0 0 0.16" rpy="${-pi/2} 0 ${-pi/2}"/>
+        <parent link="ur3_d435_mount_link"/>
+        <child link="gripper_axe"/>
+      </joint>
 </robot>
