Commit message: fix gripper and handle configurations for plaque-ur3

File: urdf/plaque-ur3.urdf (robot description, URDF)
Before this commit: robot plaque-tubes, 27 links, 26 joints
Links:
- link plaque_link: geometry collision box size=0.258 0.307 0.005; visual box size=0.258 0.307 0.005
Joints:
- joint to_hole_00: origin xyz=0 0.0275 -0.071 rpy=0 0 0 -> xyz=0.0275 -0.071 0 rpy=0 0 0
- joint to_hole_01: origin xyz= 0 0.046 -0.071 rpy=0 0 0 -> xyz=0.046 -0.071  0 rpy=0 0 0
- joint to_hole_02: origin xyz=0 0.046 -0.1145 rpy=0 0 0 -> xyz=0.046 -0.1145 0 rpy=0 0 0
- joint to_hole_03: origin xyz=0 0.0275 -0.0925 rpy=0 0 0 -> xyz=0.0275 -0.0925 0 rpy=0 0 0
- joint to_hole_04: origin xyz= 0 0.046 -0.0925 rpy=0 0 0 -> xyz= 0.046 -0.0925 0 rpy=0 0 0
- joint to_hole_05: origin xyz=0 0.0275 -0.1145 rpy=0 0 0 -> xyz=0.0275 -0.1145 0 rpy=0 0 0
- joint to_hole_06: origin xyz=0 0.2125 -0.071 rpy=0 0 0 -> xyz= 0.2125 -0.071 0 rpy=0 0 0
- joint to_hole_07: origin xyz=0 0.231 -0.071 rpy=0 0 0 -> xyz=0.231 -0.071 0 rpy=0 0 0
- joint to_hole_08: origin xyz=0 0.2125 -0.0925 rpy=0 0 0 -> xyz=0.2125 -0.0925 0 rpy=0 0 0
- joint to_hole_09: origin xyz=0 0.231 -0.0925 rpy=0 0 0 -> xyz=0.231 -0.0925 0 rpy=0 0 0
- joint to_hole_10: origin xyz=0 0.2125 -0.1145 rpy=0 0 0 -> xyz=0.2125 -0.1145 0 rpy=0 0 0
- joint to_hole_11: origin xyz=0 0.231 -0.1145 rpy=0 0 0 -> xyz=0.231 -0.1145 0 rpy=0 0 0
- joint to_hole_12: origin xyz=0 0.0275 -0.192 rpy=0 0 0 -> xyz=0.0275 -0.192 0 rpy=0 0 0
- joint to_hole_13: origin xyz=0 0.046 -0.192 rpy=0 0 0 -> xyz=0.046 -0.192 0 rpy=0 0 0
- joint to_hole_14: origin xyz=0 0.0275 -0.2135 rpy=0 0 0 -> xyz=0.0275 -0.2135 0 rpy=0 0 0
- joint to_hole_15: origin xyz=0 0.046 -0.2135 rpy=0 0 0 -> xyz=0.046 -0.2135 0 rpy=0 0 0
- joint to_hole_16: origin xyz=0 0.0275 -0.2355 rpy=0 0 0 -> xyz=0.0275 -0.2355 0 rpy=0 0 0
- joint to_hole_17: origin xyz=0 0.046 -0.2355 rpy=0 0 0 -> xyz=0.046 -0.2355 0 rpy=0 0 0
- joint to_hole_18: origin xyz=0 0.2125 -0.192 rpy=0 0 0 -> xyz=0.2125 -0.192 0 rpy=0 0 0
- joint to_hole_19: origin xyz=0 0.231 -0.192 rpy=0 0 0 -> xyz=0.231 -0.192 0 rpy=0 0 0
- joint to_hole_20: origin xyz=0 0.2125 -0.2135 rpy=0 0 0 -> xyz=0.2125 -0.2135 0 rpy=0 0 0
- joint to_hole_21: origin xyz=0 0.231 -0.2135 rpy=0 0 0 -> xyz=0.231 -0.2135 0 rpy=0 0 0
- joint to_hole_22: origin xyz=0 0.2125 -0.2355 rpy=0 0 0 -> xyz=0.2125 -0.2355 0 rpy=0 0 0
- joint to_hole_23: origin xyz=0 0.231 -0.2355 rpy=0 0 0 -> xyz=0.231 -0.2355 0 rpy=0 0 0

Commit message: add nuts and screws models

File: urdf/plaque-ur3.urdf (robot description, URDF)
Before this commit: robot plaque-tubes, 27 links, 26 joints
Links:
- added link nut_01_link; visual cylinder length=0.007 radius=0.00135
- added link nut_02_link; visual cylinder length=0.007 radius=0.00135
- added link nut_03_link; visual cylinder length=0.007 radius=0.00135
- added link screw_00_link; visual cylinder length=0.008 radius=0.00125
- added link screw_01_link; visual cylinder length=0.008 radius=0.00125
- added link screw_02_link; visual cylinder length=0.008 radius=0.00125
- added link screw_03_link; visual cylinder length=0.008 radius=0.00125
- added link screw_04_link; visual cylinder length=0.008 radius=0.00125
- added link screw_05_link; visual cylinder length=0.008 radius=0.00125
- added link screw_06_link; visual cylinder length=0.008 radius=0.00125
- added link screw_07_link; visual cylinder length=0.008 radius=0.00125
- added link screw_08_link; visual cylinder length=0.008 radius=0.00125
- added link screw_09_link; visual cylinder length=0.008 radius=0.00125
- added link screw_10_link; visual cylinder length=0.008 radius=0.00125
- added link screw_11_link; visual cylinder length=0.008 radius=0.00125
Joints:
- added joint to_nut_01: type fixed, parent plaque_link, child nut_01_link, origin xyz=0.129 -0.079 0 rpy=0 0 0
- added joint to_nut_02: type fixed, parent plaque_link, child nut_02_link, origin xyz=0.129 -0.1535 0 rpy=0 0 0
- added joint to_nut_03: type fixed, parent plaque_link, child nut_03_link, origin xyz=0.129 -0.228 0 rpy=0 0 0
- added joint to_screw_00: type fixed, parent plaque_link, child screw_00_link, origin xyz=0.104 -0.256 0 rpy=0 0 0
- added joint to_screw_01: type fixed, parent plaque_link, child screw_01_link, origin xyz=0.129 -0.256 0 rpy=0 0 0
- added joint to_screw_02: type fixed, parent plaque_link, child screw_02_link, origin xyz=0.1585 -0.256 0 rpy=0 0 0
- added joint to_screw_03: type fixed, parent plaque_link, child screw_03_link, origin xyz=0.179 -0.256 0 rpy=0 0 0
- added joint to_screw_04: type fixed, parent plaque_link, child screw_04_link, origin xyz=0.204 -0.256 0 rpy=0 0 0
- added joint to_screw_05: type fixed, parent plaque_link, child screw_05_link, origin xyz=0.229 -0.256 0 rpy=0 0 0
- added joint to_screw_06: type fixed, parent plaque_link, child screw_06_link, origin xyz=0.104 -0.2725 0 rpy=0 0 0
- added joint to_screw_07: type fixed, parent plaque_link, child screw_07_link, origin xyz=0.129 -0.2725 0 rpy=0 0 0
- added joint to_screw_08: type fixed, parent plaque_link, child screw_08_link, origin xyz=0.1585 -0.2725 0 rpy=0 0 0
- added joint to_screw_09: type fixed, parent plaque_link, child screw_09_link, origin xyz=0.179 -0.2725 0 rpy=0 0 0
- added joint to_screw_10: type fixed, parent plaque_link, child screw_10_link, origin xyz=0.204 -0.2725 0 rpy=0 0 0
- added joint to_screw_11: type fixed, parent plaque_link, child screw_11_link, origin xyz=0.229 -0.2725 0 rpy=0 0 0
