Commit message: demo pick and place UR3

File: urdf/plaque-ur3.urdf (robot description, URDF)
Before this commit: robot plaque-tubes, 42 links, 41 joints
Links:
- removed link hole_00_link
- removed link hole_01_link
- removed link hole_02_link
- removed link hole_03_link
- removed link hole_04_link
- removed link hole_05_link
- removed link hole_06_link
- removed link hole_07_link
- removed link hole_08_link
- removed link hole_09_link
- removed link hole_10_link
- removed link hole_11_link
- removed link hole_12_link
- removed link hole_13_link
- removed link hole_14_link
- removed link hole_15_link
- removed link hole_16_link
- removed link hole_17_link
- removed link hole_18_link
- removed link hole_19_link
- removed link hole_20_link
- removed link hole_21_link
- removed link hole_22_link
- removed link hole_23_link
- removed link nut_01_link
- removed link nut_02_link
- removed link nut_03_link
- removed link screw_00_link
- removed link screw_01_link
- removed link screw_02_link
- removed link screw_03_link
- removed link screw_04_link
- removed link screw_05_link
- removed link screw_06_link
- removed link screw_07_link
- removed link screw_08_link
- removed link screw_09_link
- removed link screw_10_link
- removed link screw_11_link
- added link handle_00_link
- added link handle_01_link
- added link handle_02_link
- added link handle_03_link
- added link handle_04_link
- added link handle_05_link
- added link handle_06_link
- added link handle_07_link
- added link handle_08_link
- added link handle_09_link
- added link handle_10_link
- added link handle_11_link
- added link handle_12_link
- added link handle_13_link
- added link handle_14_link
- added link handle_15_link
- added link handle_16_link
- added link handle_17_link
- added link handle_18_link
- added link handle_19_link
- added link handle_20_link
- added link handle_21_link
- added link handle_22_link
- added link handle_23_link
- added link handle_24_link
- added link handle_25_link
- added link handle_26_link
- added link handle_27_link
- added link handle_28_link
- added link handle_29_link
- added link handle_30_link
- added link handle_31_link
- added link handle_32_link
- added link handle_33_link
- added link handle_34_link
- added link handle_35_link
- added link handle_36_link
- added link handle_37_link
- added link handle_38_link
- added link handle_39_link
- added link handle_40_link
- added link handle_41_link
- added link handle_42_link
- added link handle_43_link
- added link handle_44_link
- added link handle_45_link
- added link handle_46_link
- added link handle_47_link
- added link handle_48_link
- added link handle_49_link
- added link handle_50_link
- added link handle_51_link
- added link handle_52_link
- added link handle_53_link
- added link handle_54_link
- added link handle_55_link
- added link handle_56_link
- added link handle_57_link
- added link handle_58_link
- added link handle_59_link
- added link handle_60_link
- added link handle_61_link
- added link handle_62_link
- added link handle_63_link
- added link handle_64_link
- added link handle_65_link
- added link handle_66_link
- added link handle_67_link
- added link handle_68_link
- added link handle_69_link
- added link handle_70_link
- added link handle_71_link
- added link handle_72_link
- added link handle_73_link
- added link handle_74_link
- added link handle_75_link
- added link handle_76_link
- added link handle_77_link
- added link handle_78_link
- added link handle_79_link
- added link handle_80_link
- added link handle_81_link
- added link handle_82_link
- added link handle_83_link
- added link handle_84_link
- added link handle_85_link
- added link handle_86_link
- added link handle_87_link
- added link handle_88_link
- added link handle_89_link
- added link handle_90_link
- added link handle_91_link
- added link handle_92_link; visual cylinder length=0.007 radius=0.00135
- added link handle_93_link; visual cylinder length=0.007 radius=0.00135
- added link handle_94_link; visual cylinder length=0.007 radius=0.00135
- link plaque_link: geometry collision mesh filename=package://agimus_demos/ur3/pointing/meshes/plaque.stl scale=0.001 0.001 0.001; visual mesh filename=package://agimus_demos/ur3/pointing/meshes/plaque.stl scale=0.001 0.001 0.001
Joints:
- removed joint to_hole_00
- removed joint to_hole_01
- removed joint to_hole_02
- removed joint to_hole_03
- removed joint to_hole_04
- removed joint to_hole_05
- removed joint to_hole_06
- removed joint to_hole_07
- removed joint to_hole_08
- removed joint to_hole_09
- removed joint to_hole_10
- removed joint to_hole_11
- removed joint to_hole_12
- removed joint to_hole_13
- removed joint to_hole_14
- removed joint to_hole_15
- removed joint to_hole_16
- removed joint to_hole_17
- removed joint to_hole_18
- removed joint to_hole_19
- removed joint to_hole_20
- removed joint to_hole_21
- removed joint to_hole_22
- removed joint to_hole_23
- removed joint to_nut_01
- removed joint to_nut_02
- removed joint to_nut_03
- removed joint to_screw_00
- removed joint to_screw_01
- removed joint to_screw_02
- removed joint to_screw_03
- removed joint to_screw_04
- removed joint to_screw_05
- removed joint to_screw_06
- removed joint to_screw_07
- removed joint to_screw_08
- removed joint to_screw_09
- removed joint to_screw_10
- removed joint to_screw_11
- added joint to_handle_00: type fixed, parent plaque_link, child handle_00_link, origin xyz=0.027 -0.071 0 rpy=0 0 0
- added joint to_handle_01: type fixed, parent plaque_link, child handle_01_link, origin xyz=0.046 -0.071 0 rpy=0 0 0
- added joint to_handle_02: type fixed, parent plaque_link, child handle_02_link, origin xyz=0.0645 -0.071 0 rpy=0 0 0
- added joint to_handle_03: type fixed, parent plaque_link, child handle_03_link, origin xyz=0.083 -0.071 0 rpy=0 0 0
- added joint to_handle_04: type fixed, parent plaque_link, child handle_04_link, origin xyz=0.1015 -0.071 0 rpy=0 0 0
- added joint to_handle_05: type fixed, parent plaque_link, child handle_05_link, origin xyz=0.12 -0.071 0 rpy=0 0 0
- added joint to_handle_06: type fixed, parent plaque_link, child handle_06_link, origin xyz=0.1385 -0.071 0 rpy=0 0 0
- added joint to_handle_07: type fixed, parent plaque_link, child handle_07_link, origin xyz=0.157 -0.071 0 rpy=0 0 0
- added joint to_handle_08: type fixed, parent plaque_link, child handle_08_link, origin xyz=0.1755 -0.071 0 rpy=0 0 0
- added joint to_handle_09: type fixed, parent plaque_link, child handle_09_link, origin xyz=0.194 -0.071 0 rpy=0 0 0
- added joint to_handle_10: type fixed, parent plaque_link, child handle_10_link, origin xyz=0.2125 -0.071 0 rpy=0 0 0
- added joint to_handle_11: type fixed, parent plaque_link, child handle_11_link, origin xyz=0.231 -0.071 0 rpy=0 0 0
- added joint to_handle_12: type fixed, parent plaque_link, child handle_12_link, origin xyz=0.027 -0.093 0 rpy=0 0 0
- added joint to_handle_13: type fixed, parent plaque_link, child handle_13_link, origin xyz=0.046 -0.093 0 rpy=0 0 0
- added joint to_handle_14: type fixed, parent plaque_link, child handle_14_link, origin xyz=0.0645 -0.093 0 rpy=0 0 0
- added joint to_handle_15: type fixed, parent plaque_link, child handle_15_link, origin xyz=0.083 -0.093 0 rpy=0 0 0
- added joint to_handle_16: type fixed, parent plaque_link, child handle_16_link, origin xyz=0.1015 -0.093 0 rpy=0 0 0
- added joint to_handle_17: type fixed, parent plaque_link, child handle_17_link, origin xyz=0.12 -0.093 0 rpy=0 0 0
- added joint to_handle_18: type fixed, parent plaque_link, child handle_18_link, origin xyz=0.1385 -0.093 0 rpy=0 0 0
- added joint to_handle_19: type fixed, parent plaque_link, child handle_19_link, origin xyz=0.157 -0.093 0 rpy=0 0 0
- added joint to_handle_20: type fixed, parent plaque_link, child handle_20_link, origin xyz=0.1755 -0.093 0 rpy=0 0 0
- added joint to_handle_21: type fixed, parent plaque_link, child handle_21_link, origin xyz=0.194 -0.093 0 rpy=0 0 0
- added joint to_handle_22: type fixed, parent plaque_link, child handle_22_link, origin xyz=0.2125 -0.093 0 rpy=0 0 0
- added joint to_handle_23: type fixed, parent plaque_link, child handle_23_link, origin xyz=0.231 -0.093 0 rpy=0 0 0
- added joint to_handle_24: type fixed, parent plaque_link, child handle_24_link, origin xyz=0.027 -0.115 0 rpy=0 0 0
- added joint to_handle_25: type fixed, parent plaque_link, child handle_25_link, origin xyz=0.046 -0.115 0 rpy=0 0 0
- added joint to_handle_26: type fixed, parent plaque_link, child handle_26_link, origin xyz=0.0645 -0.115 0 rpy=0 0 0
- added joint to_handle_27: type fixed, parent plaque_link, child handle_27_link, origin xyz=0.083 -0.115 0 rpy=0 0 0
- added joint to_handle_28: type fixed, parent plaque_link, child handle_28_link, origin xyz=0.1385 -0.115 0 rpy=0 0 0
- added joint to_handle_29: type fixed, parent plaque_link, child handle_29_link, origin xyz=0.157 -0.115 0 rpy=0 0 0
- added joint to_handle_30: type fixed, parent plaque_link, child handle_30_link, origin xyz=0.1755 -0.115 0 rpy=0 0 0
- added joint to_handle_31: type fixed, parent plaque_link, child handle_31_link, origin xyz=0.194 -0.115 0 rpy=0 0 0
- added joint to_handle_32: type fixed, parent plaque_link, child handle_32_link, origin xyz=0.2125 -0.115 0 rpy=0 0 0
- added joint to_handle_33: type fixed, parent plaque_link, child handle_33_link, origin xyz=0.231 -0.115 0 rpy=0 0 0
- added joint to_handle_34: type fixed, parent plaque_link, child handle_34_link, origin xyz=0.027 -0.192 0 rpy=0 0 0
- added joint to_handle_35: type fixed, parent plaque_link, child handle_35_link, origin xyz=0.046 -0.192 0 rpy=0 0 0
- added joint to_handle_36: type fixed, parent plaque_link, child handle_36_link, origin xyz=0.0645 -0.192 0 rpy=0 0 0
- added joint to_handle_37: type fixed, parent plaque_link, child handle_37_link, origin xyz=0.083 -0.192 0 rpy=0 0 0
- added joint to_handle_38: type fixed, parent plaque_link, child handle_38_link, origin xyz=0.1015 -0.192 0 rpy=0 0 0
- added joint to_handle_39: type fixed, parent plaque_link, child handle_39_link, origin xyz=0.12 -0.192 0 rpy=0 0 0
- added joint to_handle_40: type fixed, parent plaque_link, child handle_40_link, origin xyz=0.1755 -0.192 0 rpy=0 0 0
- added joint to_handle_41: type fixed, parent plaque_link, child handle_41_link, origin xyz=0.194 -0.192 0 rpy=0 0 0
- added joint to_handle_42: type fixed, parent plaque_link, child handle_42_link, origin xyz=0.2125 -0.192 0 rpy=0 0 0
- added joint to_handle_43: type fixed, parent plaque_link, child handle_43_link, origin xyz=0.231 -0.192 0 rpy=0 0 0
- added joint to_handle_44: type fixed, parent plaque_link, child handle_44_link, origin xyz=0.027 -0.214 0 rpy=0 0 0
- added joint to_handle_45: type fixed, parent plaque_link, child handle_45_link, origin xyz=0.046 -0.214 0 rpy=0 0 0
- added joint to_handle_46: type fixed, parent plaque_link, child handle_46_link, origin xyz=0.0645 -0.214 0 rpy=0 0 0
- added joint to_handle_47: type fixed, parent plaque_link, child handle_47_link, origin xyz=0.083 -0.214 0 rpy=0 0 0
- added joint to_handle_48: type fixed, parent plaque_link, child handle_48_link, origin xyz=0.1015 -0.214 0 rpy=0 0 0
- added joint to_handle_49: type fixed, parent plaque_link, child handle_49_link, origin xyz=0.12 -0.214 0 rpy=0 0 0
- added joint to_handle_50: type fixed, parent plaque_link, child handle_50_link, origin xyz=0.1385 -0.214 0 rpy=0 0 0
- added joint to_handle_51: type fixed, parent plaque_link, child handle_51_link, origin xyz=0.157 -0.214 0 rpy=0 0 0
- added joint to_handle_52: type fixed, parent plaque_link, child handle_52_link, origin xyz=0.1755 -0.214 0 rpy=0 0 0
- added joint to_handle_53: type fixed, parent plaque_link, child handle_53_link, origin xyz=0.194 -0.214 0 rpy=0 0 0
- added joint to_handle_54: type fixed, parent plaque_link, child handle_54_link, origin xyz=0.2125 -0.214 0 rpy=0 0 0
- added joint to_handle_55: type fixed, parent plaque_link, child handle_55_link, origin xyz=0.231 -0.214 0 rpy=0 0 0
- added joint to_handle_56: type fixed, parent plaque_link, child handle_56_link, origin xyz=0.027 -0.236 0 rpy=0 0 0
- added joint to_handle_57: type fixed, parent plaque_link, child handle_57_link, origin xyz=0.046 -0.236 0 rpy=0 0 0
- added joint to_handle_58: type fixed, parent plaque_link, child handle_58_link, origin xyz=0.0645 -0.236 0 rpy=0 0 0
- added joint to_handle_59: type fixed, parent plaque_link, child handle_59_link, origin xyz=0.083 -0.236 0 rpy=0 0 0
- added joint to_handle_60: type fixed, parent plaque_link, child handle_60_link, origin xyz=0.1015 -0.236 0 rpy=0 0 0
- added joint to_handle_61: type fixed, parent plaque_link, child handle_61_link, origin xyz=0.12 -0.236 0 rpy=0 0 0
- added joint to_handle_62: type fixed, parent plaque_link, child handle_62_link, origin xyz=0.1385 -0.236 0 rpy=0 0 0
- added joint to_handle_63: type fixed, parent plaque_link, child handle_63_link, origin xyz=0.157 -0.236 0 rpy=0 0 0
- added joint to_handle_64: type fixed, parent plaque_link, child handle_64_link, origin xyz=0.1755 -0.236 0 rpy=0 0 0
- added joint to_handle_65: type fixed, parent plaque_link, child handle_65_link, origin xyz=0.194 -0.236 0 rpy=0 0 0
- added joint to_handle_66: type fixed, parent plaque_link, child handle_66_link, origin xyz=0.2125 -0.236 0 rpy=0 0 0
- added joint to_handle_67: type fixed, parent plaque_link, child handle_67_link, origin xyz=0.231 -0.236 0 rpy=0 0 0
- added joint to_handle_68: type fixed, parent plaque_link, child handle_68_link, origin xyz=0.029 -0.0265 0 rpy=0 0 0
- added joint to_handle_69: type fixed, parent plaque_link, child handle_69_link, origin xyz=0.05 -0.0265 0 rpy=0 0 0
- added joint to_handle_70: type fixed, parent plaque_link, child handle_70_link, origin xyz=0.079 -0.0265 0 rpy=0 0 0
- added joint to_handle_71: type fixed, parent plaque_link, child handle_71_link, origin xyz=0.104 -0.0265 0 rpy=0 0 0
- added joint to_handle_72: type fixed, parent plaque_link, child handle_72_link, origin xyz=0.139 -0.0265 0 rpy=0 0 0
- added joint to_handle_73: type fixed, parent plaque_link, child handle_73_link, origin xyz=0.154 -0.0265 0 rpy=0 0 0
- added joint to_handle_74: type fixed, parent plaque_link, child handle_74_link, origin xyz=0.029 -0.049 0 rpy=0 0 0
- added joint to_handle_75: type fixed, parent plaque_link, child handle_75_link, origin xyz=0.05 -0.049 0 rpy=0 0 0
- added joint to_handle_76: type fixed, parent plaque_link, child handle_76_link, origin xyz=0.079 -0.049 0 rpy=0 0 0
- added joint to_handle_77: type fixed, parent plaque_link, child handle_77_link, origin xyz=0.104 -0.049 0 rpy=0 0 0
- added joint to_handle_78: type fixed, parent plaque_link, child handle_78_link, origin xyz=0.139 -0.049 0 rpy=0 0 0
- added joint to_handle_79: type fixed, parent plaque_link, child handle_79_link, origin xyz=0.154 -0.049 0 rpy=0 0 0
- added joint to_handle_80: type fixed, parent plaque_link, child handle_80_link, origin xyz=0.1035 -0.258 0 rpy=0 0 0
- added joint to_handle_81: type fixed, parent plaque_link, child handle_81_link, origin xyz=0.129 -0.258 0 rpy=0 0 0
- added joint to_handle_82: type fixed, parent plaque_link, child handle_82_link, origin xyz=0.154 -0.258 0 rpy=0 0 0
- added joint to_handle_83: type fixed, parent plaque_link, child handle_83_link, origin xyz=0.179 -0.257 0 rpy=0 0 0
- added joint to_handle_84: type fixed, parent plaque_link, child handle_84_link, origin xyz=0.204 -0.257 0 rpy=0 0 0
- added joint to_handle_85: type fixed, parent plaque_link, child handle_85_link, origin xyz=0.229 -0.257 0 rpy=0 0 0
- added joint to_handle_86: type fixed, parent plaque_link, child handle_86_link, origin xyz=0.1035 -0.285 0 rpy=0 0 0
- added joint to_handle_87: type fixed, parent plaque_link, child handle_87_link, origin xyz=0.129 -0.285 0 rpy=0 0 0
- added joint to_handle_88: type fixed, parent plaque_link, child handle_88_link, origin xyz=0.154 -0.284 0 rpy=0 0 0
- added joint to_handle_89: type fixed, parent plaque_link, child handle_89_link, origin xyz=0.179 -0.279 0 rpy=0 0 0
- added joint to_handle_90: type fixed, parent plaque_link, child handle_90_link, origin xyz=0.204 -0.278 0 rpy=0 0 0
- added joint to_handle_91: type fixed, parent plaque_link, child handle_91_link, origin xyz=0.229 -0.278 0 rpy=0 0 0
- added joint to_handle_92: type fixed, parent plaque_link, child handle_92_link, origin xyz=0.027 -0.1535 0 rpy=0 0 0
- added joint to_handle_93: type fixed, parent plaque_link, child handle_93_link, origin xyz=0.083 -0.1535 0 rpy=0 0 0
- added joint to_handle_94: type fixed, parent plaque_link, child handle_94_link, origin xyz=0.1755 -0.1535 0 rpy=0 0 0

File: urdf/robot.urdf.xacro (robot description, xacro)
@@ -52,35 +52,35 @@
    <link name="world" />
     <link name="support_link">
-      <inertial>
-        <mass value="200"/>
-	<origin xyz="0 0 0.44"/>
-        <inertia ixx="50"  ixy="0"  ixz="0" iyy="50" iyz="0" izz="50" />
-      </inertial>
-      <!-- table -->
-      <visual>
-	<origin xyz="0.0 -0.305 0.5"/>
-        <geometry>
-	        <box size="0.80 1 1"/>
-        </geometry>
-      </visual>
-      <collision>
-        <origin xyz="0.0 -0.305 0.5"/>
-        <geometry>
-	        <box size="0.80 1 1"/>
-        </geometry>
-      </collision>
-      <!-- support -->
-     <visual>
-       <origin xyz="0 0 1.01"/>
-       <geometry>
-	        <box size="0.16 0.16 0.02"/>
-       </geometry>
-     </visual>
-     <collision>
-       <origin xyz="0 0 1.01"/>
-       <geometry>
-	        <box size="0.16 0.16 0.02"/>
-       </geometry>
-     </collision>
+        <inertial>
+            <mass value="200"/>
+        	<origin xyz="0 0 0.44"/>
+            <inertia ixx="50"  ixy="0"  ixz="0" iyy="50" iyz="0" izz="50" />
+        </inertial>
+        <!-- table -->
+            <visual>
+        	<origin xyz="0.0 -0.305 0.5"/>
+                <geometry>
+        	        <box size="0.80 1 1"/>
+                </geometry>
+              </visual>
+              <collision>
+                <origin xyz="0.0 -0.305 0.5"/>
+                <geometry>
+        	        <box size="0.80 1 1"/>
+                </geometry>
+              </collision>
+         <!-- support -->
+             <visual>
+               <origin xyz="0 0 1.01"/>
+               <geometry>
+        	        <box size="0.16 0.16 0.02"/>
+               </geometry>
+             </visual>
+             <collision>
+               <origin xyz="0 0 1.01"/>
+               <geometry>
+        	        <box size="0.16 0.16 0.02"/>
+               </geometry>
+             </collision>
     </link>
      <link name="walls">
@@ -145,5 +145,5 @@
      <parent link="support_link" />
      <child link = "walls" />
-      <origin xyz="0.0 0.0 1" rpy="0.0 0.0 0" />
+     <origin xyz="0.0 0.0 1" rpy="0.0 0.0 0" />
    </joint>
    <joint name="support_joint" type="fixed">
@@ -252,13 +252,5 @@
    <xacro:sensor_d435 parent="ref_camera_link" name="camera" use_nominal_extrinsics="true">
      <!-- <origin xyz="0 0.115 0" rpy="0 -1.0472 -1.57079632679"/> -->
-      <origin xyz="0 0 0" rpy="0 0 0"/>
+     <origin xyz="0 0 0" rpy="0 0 0"/>
    </xacro:sensor_d435>
-      <!-- Axes -->
-      <link name="gripper_axe">
-      </link>
-       <joint name="gripper_axe_joint" type="fixed">
-        <origin xyz="0 0 0.16" rpy="${-pi/2} 0 ${-pi/2}"/>
-        <parent link="ur3_d435_mount_link"/>
-        <child link="gripper_axe"/>
-      </joint>
 </robot>
