Commit message: fix files corrupted 2

File: data-simulation/robot.urdf (robot description, URDF)
Before this commit: robot ur3e, 30 links, 29 joints
Links:
- removed link ur3e_d435_mount_link
- removed link ur3e_tool_link
- removed link ur3e_tooltip_link
- added link ur3_d435_mount_link, mass 0.1; collision mesh filename=package://agimus_demos/meshes/ur3_d435_mount.stl; visual mesh filename=package://agimus_demos/meshes/ur3_d435_mount.stl
- added link ur3_tool_link, mass 0.1; collision cylinder length=0.25 radius=0.0015; collision mesh filename=package://agimus_demos/meshes/ur3_tip.stl
- added link ur3_tooltip_link
- link base_link_inertia: geometry collision mesh filename=package://ur_description/meshes/ur3/collision/base.stl; visual mesh filename=package://ur_description/meshes/ur3/visual/base.dae
- link forearm_link: geometry collision mesh filename=package://ur_description/meshes/ur3/collision/forearm.stl; visual mesh filename=package://ur_description/meshes/ur3/visual/forearm.dae
- link shoulder_link: geometry collision mesh filename=package://ur_description/meshes/ur3/collision/shoulder.stl; visual mesh filename=package://ur_description/meshes/ur3/visual/shoulder.dae
- link upper_arm_link: geometry collision mesh filename=package://ur_description/meshes/ur3/collision/upperarm.stl; visual mesh filename=package://ur_description/meshes/ur3/visual/upperarm.dae
- link wrist_1_link: geometry collision mesh filename=package://ur_description/meshes/ur3/collision/wrist1.stl; visual mesh filename=package://ur_description/meshes/ur3/visual/wrist1.dae
- link wrist_2_link: geometry collision mesh filename=package://ur_description/meshes/ur3/collision/wrist2.stl; visual mesh filename=package://ur_description/meshes/ur3/visual/wrist2.dae
- link wrist_3_link: geometry collision mesh filename=package://ur_description/meshes/ur3/collision/wrist3.stl; visual mesh filename=package://ur_description/meshes/ur3/visual/wrist3.dae
Joints:
- removed joint ur3e_d435_mount_joint
- removed joint ur3e_tool_joint
- removed joint ur3e_tooltip_joint
- added joint ur3_d435_mount_joint: type fixed, parent wrist_3_link, child ur3_d435_mount_link, origin xyz=0.0 0.0 0.0 rpy=0.0 0.0 3.14159265359
- added joint ur3_tool_joint: type fixed, parent ur3_d435_mount_link, child ur3_tool_link, origin xyz=0.0000 0.0000 0.0 rpy=0.0 0.0 0.0
- added joint ur3_tooltip_joint: type fixed, parent ur3_tool_link, child ur3_tooltip_link, origin xyz=0.0 0.0 0.25 rpy=0.0 0.0 0.0
- joint ref_camera_joint: parent ur3e_d435_mount_link -> ur3_d435_mount_link

File: urdf/april-tag-plank.urdf (robot description, URDF)
Before this commit: robot plank-with-april-tags, 1 links, 0 joints
Links:
- link base_link: geometry visual box size=0.21 0.297 0.005

File: urdf/plaque-ur3.urdf (robot description, URDF)
Before this commit: robot plaque-tubes, 42 links, 41 joints
Links:
- link plaque_link: geometry visual box size=0.258 0.307 0.005

File: urdf/robot-init.urdf.xacro (robot description, xacro)
@@ -1,4 +1,4 @@
 <?xml version="1.0"?>
-<robot xmlns:xacro="http://wiki.ros.org/xacro" name="ur3e" >
+<robot xmlns:xacro="http://wiki.ros.org/xacro" name="ur3" >
   <material name="white02">
     <color rgba="1 1 1 0.2"/>
@@ -8,11 +8,11 @@
              doc="whether robot is loaded in gazebo simulator"/>
   <xacro:arg name="joint_limit_params"
-             default="$(find ur_description)/config/ur3e/joint_limits.yaml"/>
+             default="$(find ur_description)/config/ur3/joint_limits.yaml"/>
   <xacro:arg name="kinematics_params"
              default="$(find agimus_demos)/ur3/pointing/config/calibrated-params.yaml"/>
   <xacro:arg name="physical_params"
-             default="$(find ur_description)/config/ur3e/physical_parameters.yaml"/>
+             default="$(find ur_description)/config/ur3/physical_parameters.yaml"/>
   <xacro:arg name="visual_params"
-             default="$(find ur_description)/config/ur3e/visual_parameters.yaml"/>
+             default="$(find ur_description)/config/ur3/visual_parameters.yaml"/>
   <!-- legal values:
        - hardware_interface/PositionJointInterface
@@ -203,5 +203,5 @@
      </visual> -->
    </link>
-   <link name="ur3e_d435_mount_link">
+   <link name="ur3_d435_mount_link">
      <inertial>
        <origin xyz="0.0 0.0 0.0" rpy="0 0 0" />
@@ -214,5 +214,5 @@
        <origin xyz="0 0 0" rpy="0 0 0" />
        <geometry>
-         <mesh filename="package://agimus_demos/ur3/pointing/meshes/ur3e_d435_mount.stl"/>
+         <mesh filename="package://agimus_demos/ur3/pointing/meshes/ur3_d435_mount.stl"/>
        </geometry>
        <material name="Red">
@@ -223,14 +223,14 @@
        <origin xyz="0 0 0" rpy="0 0 0" />
        <geometry>
-         <mesh filename="package://agimus_demos/ur3/pointing/meshes/ur3e_d435_mount.stl"/>
-       </geometry>
-     </collision>
-   </link>
-   <joint name="ur3e_d435_mount_joint" type="fixed">
+         <mesh filename="package://agimus_demos/ur3/pointing/meshes/ur3_d435_mount.stl"/>
+       </geometry>
+     </collision>
+   </link>
+   <joint name="ur3_d435_mount_joint" type="fixed">
      <parent link="wrist_3_link"/>
-     <child link="ur3e_d435_mount_link" />
+     <child link="ur3_d435_mount_link" />
      <origin xyz="0.0 0.0 0.0" rpy="0.0 0.0 3.14159265359" />
    </joint>
-   <link name="ur3e_tool_link">
+   <link name="ur3_tool_link">
      <inertial>
        <origin xyz="0.0 0.0 0.0" rpy="0 0 0" />
@@ -244,5 +244,5 @@
        <origin xyz="0 0 0" rpy="0 0 0" />
        <geometry>
-         <mesh filename="package://agimus_demos/ur3/pointing/meshes/ur3e_tip.stl"/>
+         <mesh filename="package://agimus_demos/ur3/pointing/meshes/ur3_tip.stl"/>
        </geometry>
        <material name="Red">
@@ -253,5 +253,5 @@
        <origin xyz="0 0 0" rpy="0 0 0" />
        <geometry>
-         <mesh filename="package://agimus_demos/ur3/pointing/meshes/ur3e_tip.stl"/>
+         <mesh filename="package://agimus_demos/ur3/pointing/meshes/ur3_tip.stl"/>
        </geometry>
      </collision>
@@ -273,14 +273,14 @@
      </collision>
    </link>
-   <joint name="ur3e_tool_joint" type="fixed">
-     <parent link="ur3e_d435_mount_link"/>
-     <child link="ur3e_tool_link" />
+   <joint name="ur3_tool_joint" type="fixed">
+     <parent link="ur3_d435_mount_link"/>
+     <child link="ur3_tool_link" />
      <origin xyz="$(arg tip_offset_x) $(arg tip_offset_y) 0.0" rpy="0.0 0.0 0.0" />
    </joint>
-   <link name="ur3e_tooltip_link">
-   </link>
-  <joint name="ur3e_tooltip_joint" type="fixed">
-     <parent link="ur3e_tool_link" />
-     <child link = "ur3e_tooltip_link" />
+   <link name="ur3_tooltip_link">
+   </link>
+  <joint name="ur3_tooltip_joint" type="fixed">
+     <parent link="ur3_tool_link" />
+     <child link = "ur3_tooltip_link" />
      <origin xyz="0.0 0.0 ${0.25 + $(arg tip_offset_z)}" rpy="0.0 0.0 0.0" />
   </joint>
@@ -288,5 +288,5 @@
    </link>
     <joint name="ref_camera_joint" type="fixed">
-     <parent link="ur3e_d435_mount_link" />
+     <parent link="ur3_d435_mount_link" />
      <child link = "ref_camera_link" />
      <origin xyz="${camera_pose['camera']['x']}

File: urdf/robot.urdf.xacro (robot description, xacro)
@@ -1,4 +1,4 @@
 <?xml version="1.0"?>
-<robot xmlns:xacro="http://wiki.ros.org/xacro" name="ur3e" >
+<robot xmlns:xacro="http://wiki.ros.org/xacro" name="ur3" >
   <material name="white02">
     <color rgba="1 1 1 0.2"/>
@@ -8,11 +8,11 @@
              doc="whether robot is loaded in gazebo simulator"/>
   <xacro:arg name="joint_limit_params"
-             default="$(find ur_description)/config/ur3e/joint_limits.yaml"/>
+             default="$(find ur_description)/config/ur3/joint_limits.yaml"/>
   <xacro:arg name="kinematics_params"
              default="$(find agimus_demos)/ur3/pointing/config/calibrated-params.yaml"/>
   <xacro:arg name="physical_params"
-             default="$(find ur_description)/config/ur3e/physical_parameters.yaml"/>
+             default="$(find ur_description)/config/ur3/physical_parameters.yaml"/>
   <xacro:arg name="visual_params"
-             default="$(find ur_description)/config/ur3e/visual_parameters.yaml"/>
+             default="$(find ur_description)/config/ur3/visual_parameters.yaml"/>
   <!-- legal values:
        - hardware_interface/PositionJointInterface
@@ -85,21 +85,4 @@
     </link>
      <link name="walls">
-<<<<<<< HEAD
-     <!-- front wall -->
-     <!-- visual -->
-	<!-- origin xyz="0.385 -0.305 0.37"/ -->
-        <!-- geometry -->
-	  <!-- box size="0.03 1 0.74"/ -->
-        <!-- /geometry -->
-	<!-- material name="white02"/ -->
-     <!-- /visual -->
-      <collision>
-       <origin xyz="0.385 -0.305 0.37"/>
-       <geometry>
-	 <box size="0.03 1 0.74"/>
-       </geometry>
-      </collision>
-=======
->>>>>>> e1ef91ccdd252f7603bcc3c28882b41d48d39d22
       <!-- behind wall -->
      <visual>
@@ -174,11 +157,4 @@
       <origin xyz="0.0 0.0 1" rpy="0.0 0.0 -1.5707963" />
    </joint>
-<<<<<<< HEAD
-    <link name="ee_gripper">
-      <visual>
-        <geometry>
-          <!-- The path to the visual meshes in the package. -->
-          <mesh filename="package://agimus_demos/ur3/pointing/meshes/gripper_2f85_opened.stl" scale = "0.0008 0.0008 0.0008" />
-=======
    <!-- Gripper -->
     <link name="robotiq_85_gripper">
@@ -186,26 +162,8 @@
         <geometry>
           <mesh filename="package://agimus_demos/ur3/pointing/meshes/gripper_2f85_opened.stl" scale = "0.001 0.001 0.001" />
->>>>>>> e1ef91ccdd252f7603bcc3c28882b41d48d39d22
         </geometry>
       </visual>
       <collision>
         <geometry>
-<<<<<<< HEAD
-          <!-- The path to the collision meshes in the package. -->
-          <mesh filename="package://agimus_demos/ur3/pointing/meshes/gripper_2f85_opened.stl" scale = "0.0008 0.0008 0.0008" />
-        </geometry>
-      </collision>
-    </link>
-    <joint name="ee_gripper_joint" type="fixed">
-      <!-- The parent link must be read from the robot model it is attached to. -->
-      <parent link="wrist_3_link"/>
-      <child link="ee_gripper"/>
-      <origin rpy="1.5708 0 0" xyz="0 0.075 0"/>
-    </joint>
-    <!-- TCP frame -->
-    <joint name="tcp_joint" type="fixed">
-      <origin xyz="0 0 0.116" rpy="0 0 0"/>
-      <parent link="ee_gripper"/>
-=======
           <mesh filename="package://agimus_demos/ur3/pointing/meshes/gripper_2f85_opened.stl" scale = "0.001 0.001 0.001" />
         </geometry>
@@ -232,6 +190,6 @@
   </link>
   <joint name="robotiq_coupler_joint" type="fixed">
-    <origin xyz="0 0 0.01" rpy="0 0 ${-pi/2.0}" />
-    <parent link="tool0"/>
+    <origin xyz="0 0 0.015" rpy="0 0 ${pi/2.0}" />
+    <parent link="ur3_d435_mount_link"/>
     <child link="robotiq_coupler"/>
   </joint>
@@ -240,5 +198,5 @@
      <parent link="robotiq_coupler"/>
      <child link="robotiq_85_gripper"/>
-    <origin xyz="-0.09 0 0" rpy="${pi/2} 0 ${pi/2}"/>
+    <origin xyz="-0.094 0 0" rpy="${pi/2} 0 ${pi/2}"/>
   </joint>
     <!-- TCP frame -->
@@ -246,10 +204,7 @@
       <origin xyz="0 0 0.116" rpy="0 0 0"/>
       <parent link="robotiq_85_gripper"/>
->>>>>>> e1ef91ccdd252f7603bcc3c28882b41d48d39d22
       <child link="tcp"/>
     </joint>
     <link name="tcp"/>
-<<<<<<< HEAD
-=======
     <!-- Camera -->
     <link name="ur3_d435_mount_link">
@@ -282,13 +237,8 @@
      <origin xyz="0.0 0.0 0.0" rpy="0.0 0.0 3.14159265359" />
    </joint>
->>>>>>> e1ef91ccdd252f7603bcc3c28882b41d48d39d22
    <link name="ref_camera_link">
    </link>
     <joint name="ref_camera_joint" type="fixed">
-<<<<<<< HEAD
-     <parent link="wrist_3_link" />
-=======
      <parent link="ur3_d435_mount_link" />
->>>>>>> e1ef91ccdd252f7603bcc3c28882b41d48d39d22
      <child link = "ref_camera_link" />
      <origin xyz="${camera_pose['camera']['x']}
@@ -304,7 +254,4 @@
       <origin xyz="0 0 0" rpy="0 0 0"/>
    </xacro:sensor_d435>
-<<<<<<< HEAD
-</robot>
-=======
       <!-- Axes -->
       <link name="gripper_axe">
@@ -316,3 +263,2 @@
       </joint>
 </robot>
->>>>>>> e1ef91ccdd252f7603bcc3c28882b41d48d39d22
